File: Maverick1000/kicad/SKYWARD-COMPUTE-CARRIER/SKYWARD-COMPUTE-CARRIER.kicad_pcb (KiCad board)
At the start: 4 copper layers, 110 x 90 mm, 75 parts, among them J1 CM4_J1, J10 DEBUG, J2 CM4_J2, J3 BATT_IN, J4 DOCK, J5 FC, J6 GNSS, J7 ELRS, J8 TOF, J9 TERRA, Q1 SQJ438EP, Q2 SQJ438EP, SW1 nRPIBOOT, SW2 RUN, U1 LM74610QDBVRQ1, U2 LM74610QDBVRQ1, U3 BQ25792RQMR, U4 TPS5430DDA, U5 AP2112K-3.3TRG1, U6 INA3221AIPW

Commit message: Audit SKYWARD-COMPUTE-CARRIER Rev A: verify against real datasheets, run real DRC, route priority nets, fix defects found
Full engineering audit pass per the fabrication-readiness review brief.
Re-verified every real component against authoritative sources instead of
trusting the existing netlist, and fixed what was found broken rather than
routing around it:

- CM4 J1/J2 pin numbers and footprint (DF40C-100DS-0.4V pad numbering was
  sequential instead of the real odd/even scheme -- would have produced a
  non-functional board), plus a UART-availability architecture error
  (assumed 5 independent UARTs, only 3 are actually usable)
- BQ25792 charger fully re-modeled from a fictional 8-pin part to the real
  29-pin WQFN 4-switch buck-boost topology, with a complete verified
  application circuit
- LM74610 ORing controller corrected from an invented 6-pin package to the
  real 8-pin VSSOP-8 (no GND pin, floats between ANODE/CATHODE)
- P-FET part number "SQJ438EP" was not a real, findable part; replaced
  with verified-real DMP2305U-7
- CM4 J2 schematic symbol was reusing J1's pin labels (net wiring was
  correct, displayed pin names were wrong for ~half of J2's pins) -- found
  via an ERC-equivalent netlist check, fixed with a distinct J2 symbol
- U4 (TPS5430 5V buck) was missing its catch diode entirely -- confirmed
  non-synchronous via 6 independent reference designs, fixed by adding D5

Ran real KiCad DRC (pcbnew.WriteDRCReport, since this KiCad 7.0.11 build
has no CLI erc/drc subcommands) and used it to find and fix two more real
bugs: a collision-checker bug in this project's own router that had
wrongly certified some tracks as short-free when they actually crossed a
different net, and a BQ25792 footprint exposed-pad overlapping real pins.

Routed the 59 highest-priority nets (battery/converter/charging paths)
with a verified point-to-point router: 13 succeeded as real, DRC-clean
copper; 46 remain ratsnest, including every power-converter switch node.
Zone filli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
Parts:
- added C21: 10uF, Capacitor_SMD:C_0805_2012Metric, F.Cu at (62.4, 63.0)
- added C22: 100nF, Capacitor_SMD:C_0402_1005Metric, F.Cu at (70.1, 63.0)
- added D5: SS34, Diode_SMD:D_SMA, F.Cu at (62.4, 40.5)
- added Q5: DMP2305U-7, Package_TO_SOT_SMD:SOT-23, F.Cu at (70.1, 55.5)
- added Q6: DMP2305U-7, Package_TO_SOT_SMD:SOT-23, F.Cu at (15.9, 63.0)
- added R16: 5.6k, Resistor_SMD:R_0402_1005Metric, F.Cu at (23.6, 70.5)
- added R17: 10k, Resistor_SMD:R_0402_1005Metric, F.Cu at (31.4, 70.5)
- added R18: 10k, Resistor_SMD:R_0402_1005Metric, F.Cu at (39.1, 70.5)
- added R19: 10, Resistor_SMD:R_0402_1005Metric, F.Cu at (46.9, 70.5)
- added R20: 10k, Resistor_SMD:R_0402_1005Metric, F.Cu at (54.6, 70.5)
- added R21: 10k, Resistor_SMD:R_0402_1005Metric, F.Cu at (62.4, 70.5)
- C1, C2: footprint C_1210_3225Metric -> Capacitor_SMD:C_1210_3225Metric
- C10: value 100nF -> 10uF; footprint C_0402_1005Metric -> Capacitor_SMD:C_0805_2012Metric
- C11, C12, C13, C16, C17, C18: footprint C_0402_1005Metric -> Capacitor_SMD:C_0402_1005Metric
- C14, C15, C5, C6: footprint C_0603_1608Metric -> Capacitor_SMD:C_0603_1608Metric
- C3, C4, C7, C8: footprint C_0805_2012Metric -> Capacitor_SMD:C_0805_2012Metric
- C9: value 100nF -> 1uF; footprint C_0402_1005Metric -> Capacitor_SMD:C_0603_1608Metric
- D1, D2, D4: footprint D_SMB -> Diode_SMD:D_SMB
- D3: footprint D_SMA -> Diode_SMD:D_SMA
- F1, F2, F3, F4: footprint Fuse_1206_3216Metric -> Fuse:Fuse_1206_3216Metric
- J1, J2: footprint Hirose_DF40C-100DS-0.4V -> SKYWARD_Custom:Hirose_DF40C-100DS-0.4V
- J10: footprint PinHeader_1x06_P2.54mm_Vertical -> Connector_PinHeader_2.54mm:PinHeader_1x06_P2.54mm_Vertical
- J3: footprint JST_GH_SM02B-GHS-TB_1x02-1MP_P1.25mm_Horizontal -> Connector_JST:JST_GH_SM02B-GHS-TB_1x02-1MP_P1.25mm_Horizontal
- J4: footprint JST_GH_SM03B-GHS-TB_1x03-1MP_P1.25mm_Horizontal -> Connector_JST:JST_GH_SM03B-GHS-TB_1x03-1MP_P1.25mm_Horizontal
- J5, J6: footprint JST_GH_SM06B-GHS-TB_1x06-1MP_P1.25mm_Horizontal -> Connector_JST:JST_GH_SM06B-GHS-TB_1x06-1MP_P1.25mm_Horizontal
- J7: footprint JST_GH_SM04B-GHS-TB_1x04-1MP_P1.25mm_Horizontal -> Connector_JST:JST_GH_SM04B-GHS-TB_1x04-1MP_P1.25mm_Horizontal
- J8: footprint JST_SH_SM05B-SRSS-TB_1x05-1MP_P1.00mm_Horizontal -> Connector_JST:JST_SH_SM05B-SRSS-TB_1x05-1MP_P1.00mm_Horizontal
- J9: footprint Hirose_DF13-22DP-1.25V -> SKYWARD_Custom:Hirose_DF13-22DP-1.25V
- JP1: footprint SolderJumper-3_P1.3mm_Bridged12_Pad1.0x1.5mm -> Jumper:SolderJumper-3_P1.3mm_Bridged12_Pad1.0x1.5mm
- L1, L2: footprint L_Coilcraft_XAL4020-XXX -> Inductor_SMD:L_Coilcraft_XAL4020-XXX
- LED1: footprint LED_0603_1608Metric -> LED_SMD:LED_0603_1608Metric
- MH1, MH2, MH3, MH4: footprint MountingHole_2.7mm_M2.5 -> MountingHole:MountingHole_2.7mm_M2.5
- Q1, Q2: value SQJ438EP -> DMP2305U-7; footprint SOT-23 -> Package_TO_SOT_SMD:SOT-23
- R1, R10, R11, R12, R13, R14, R15, R2, R3, R5, R7, R8, R9: footprint R_0402_1005Metric -> Resistor_SMD:R_0402_1005Metric
- R6: footprint R_0603_1608Metric -> Resistor_SMD:R_0603_1608Metric
- RSH1, RSH2, RSH3: footprint R_1206_3216Metric -> Resistor_SMD:R_1206_3216Metric
- SW1, SW2: footprint SW_SPST_B3U-1000P -> Button_Switch_SMD:SW_SPST_B3U-1000P
- TP1, TP2, TP3, TP4: footprint TestPoint_Pad_D1.5mm -> TestPoint:TestPoint_Pad_D1.5mm
- U1, U2: value LM74610QDBVRQ1 -> LM74610QDGKRQ1; footprint SOT-23-6 -> Package_SO:VSSOP-8_3.0x3.0mm_P0.65mm
- U3: footprint QFN-24-1EP_4x4mm_P0.5mm_EP2.6x2.6mm -> SKYWARD_Custom:QFN-29_L4.0-W4.0-P0.40-BQ25792RQMR
- U4: footprint TI_SO-PowerPAD-8_ThermalVias -> Package_SO:TI_SO-PowerPAD-8_ThermalVias
- U5: footprint SOT-23-5 -> Package_TO_SOT_SMD:SOT-23-5
- U6: footprint TSSOP-16_4.4x5mm_P0.65mm -> Package_SO:TSSOP-16_4.4x5mm_P0.65mm
- moved C4 54.8 mm to (15.9, 48.0)
- moved RSH1 54.8 mm to (15.9, 55.5)
- moved F4 41.6 mm to (15.9, 78.0)
- moved C7 39.5 mm to (31.4, 63.0)
- moved L2 39.5 mm to (23.6, 63.0)
- moved R3 24.4 mm to (15.9, 70.5)
- moved R5 24.4 mm to (70.1, 70.5)
- moved C10 23.2 mm to (54.6, 63.0)
- moved C8 23.2 mm to (39.1, 63.0)
- moved C9 23.2 mm to (46.9, 63.0)
- moved C18 7.75 mm to (23.6, 48.0)
- moved C3 7.75 mm to (70.1, 40.5)
- moved C5 7.75 mm to (54.6, 48.0)
- moved C6 7.75 mm to (62.4, 48.0)
- moved D3 7.75 mm to (46.9, 55.5)
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Connections:
- C10 pad 1: +3V3 -> PMID
- C16 pad 1: VCAP1 -> VCAP1_L
- C16 pad 2: GND -> VCAP1_H
- C17 pad 1: VCAP2 -> VCAP2_L
- C17 pad 2: GND -> VCAP2_H
- C7 pad 1: DOCK_OK -> VBUS_IN
- C8 pad 1: BATT_F -> SYS_NODE
- C9 pad 1: +3V3 -> REGN
- J1 pad 10: +3V3 -> (no net)
- J1 pad 11: GND -> (no net)
- J1 pad 12: UART0_TXD0 -> (no net)
- J1 pad 13: UART0_RXD0 -> GND
- J1 pad 14: UART1_TXD1 -> GND
- J1 pad 15: UART1_RXD1 -> (no net)
- J1 pad 16: GND -> (no net)
- J1 pad 17: UART2_TXD -> (no net)
- J1 pad 18: UART2_RXD -> (no net)
- J1 pad 19: UART3_TXD -> (no net)
- J1 pad 20: UART3_RXD -> EEPROM_nWP
- J1 pad 21: GND -> (no net)
- J1 pad 22: I2C0_SDA -> GND
- J1 pad 23: I2C0_SCL -> GND
- J1 pad 24: I2C1_SDA -> GPIO_CHG_INT
- J1 pad 25: I2C1_SCL -> GPIO_TERRA_B
- J1 pad 26: GND -> GPIO_TERRA_TRIG
- J1 pad 27: SPI0_SCLK -> GPIO_TERRA_A
- J1 pad 28: SPI0_MOSI -> UART5_RXD5
- J1 pad 29: SPI0_MISO -> GPIO_GNSS_PPS
- J1 pad 3: +5V0 -> (no net)
- J1 pad 30: SPI0_CE0_N -> GPIO_DOCK_DET
- J1 pad 31: GND -> UART5_TXD5
- J1 pad 32: USB2_0_DP -> GND
- J1 pad 33: USB2_0_DN -> GND
- J1 pad 34: GND -> UART3_RXD3
- J1 pad 35: GPIO_DOCK_DET -> I2C0_SCL
- J1 pad 36: GPIO_GNSS_PPS -> I2C0_SDA
- J1 pad 37: GPIO_TOF_INT -> (no net)
- J1 pad 38: GPIO_TERRA_IRQ -> SPI0_SCLK
- J1 pad 39: GPIO_TERRA_TRIG -> SPI0_CE0_N
- J1 pad 4: +5V0 -> (no net)
- J1 pad 40: GPIO_TERRA_A -> SPI0_MISO
- J1 pad 41: GPIO_TERRA_B -> (no net)
- J1 pad 42: GPIO_FC_RESET -> GND
- J1 pad 43: GPIO_FC_AUX -> GND
- J1 pad 44: GPIO_STATUS_LED -> SPI0_MOSI
- J1 pad 45: GND -> GPIO_STATUS_LED
- J1 pad 46: UART4_TXD -> GPIO_FC_RESET
- J1 pad 47: UART4_RXD -> GPIO_FC_AUX
- J1 pad 49: (no net) -> GPIO_TERRA_IRQ
- J1 pad 5: +5V0 -> (no net)
- J1 pad 50: (no net) -> GPIO_TOF_INT
- J1 pad 51: (no net) -> UART0_RXD0
- J1 pad 52: (no net) -> GND
- J1 pad 53: (no net) -> GND
- J1 pad 54: (no net) -> UART3_TXD3
- J1 pad 55: (no net) -> UART0_TXD0
- J1 pad 59: (no net) -> GND
- J1 pad 6: GND -> (no net)
- J1 pad 60: (no net) -> GND
- J1 pad 65: (no net) -> GND
- J1 pad 66: (no net) -> GND
- J1 pad 7: RUN_PG_N -> GND
- J1 pad 71: (no net) -> GND
- J1 pad 74: (no net) -> GND
- J1 pad 77: (no net) -> +5V0
- J1 pad 79: (no net) -> +5V0
- J1 pad 8: EEPROM_nWP -> GND
- J1 pad 81: (no net) -> +5V0
- J1 pad 83: (no net) -> +5V0
- J1 pad 85: (no net) -> +5V0
- J1 pad 87: (no net) -> +5V0
- J1 pad 9: nRPIBOOT -> (no net)
- J1 pad 92: (no net) -> RUN_PG
- J1 pad 93: (no net) -> nRPIBOOT
- J1 pad 98: (no net) -> GND
- J1 pad 99: (no net) -> +3V3
- J10 pad 3: UART3_TXD -> UART0_TXD0
- J10 pad 4: UART3_RXD -> UART0_RXD0
- J10 pad 6: RUN_PG_N -> RUN_PG
- J2 pad 10: GND -> (no net)
- J2 pad 13: (no net) -> GND
- J2 pad 14: (no net) -> GND
- J2 pad 19: (no net) -> GND
- J2 pad 2: +5V0 -> (no net)
- J2 pad 20: (no net) -> GND
- J2 pad 25: (no net) -> GND
- J2 pad 26: (no net) -> GND
- J2 pad 3: GND -> USB2_0_DN
- J2 pad 4: +5V0 -> (no net)
- J2 pad 5: GND -> USB2_0_DP
- J2 pad 6: +5V0 -> (no net)
- J2 pad 8: +5V0 -> GND
- J2 pad 9: GND -> (no net)
- J6 pad 3: UART1_RXD1 -> UART3_RXD3
- J6 pad 4: UART1_TXD1 -> UART3_TXD3
- J7 pad 3: UART2_RXD -> UART5_RXD5
- J7 pad 4: UART2_TXD -> UART5_TXD5
- J9 pad 10: UART4_TXD -> (no net)
- J9 pad 11: UART4_RXD -> (no net)
- L2 pad 1: CHG_SW -> SW1
- L2 pad 2: BATT_F -> SW2
- R3 pad 1: PROG -> ILIM_SET
- R8 pad 2: RUN_PG_N -> RUN_PG
- SW2 pad 1: RUN_PG_N -> RUN_PG
- U1 pad 1: BATT_F -> VCAP1_L
- U1 pad 2: GND -> Q1_GATE
- U1 pad 3: VCAP1 -> (no net)
- U1 pad 4: Q1_GATE -> BATT_F
- U1 pad 5: VBAT_MAIN_OUT -> (no net)
- U1 pad 6: (no net) -> Q1_GATE
- U2 pad 1: P1_F -> VCAP2_L
- U2 pad 2: GND -> Q2_GATE
- U2 pad 3: VCAP2 -> (no net)
- U2 pad 4: Q2_GATE -> P1_F
- U2 pad 5: VBAT_P1_OUT -> (no net)
- U2 pad 6: (no net) -> Q2_GATE
- U3 pad 1: DOCK_OK -> (no net)
- U3 pad 11: (no net) -> ACDRV1_GATE
- U3 pad 12: (no net) -> QON_N
- U3 pad 13: (no net) -> GND
- U3 pad 14: (no net) -> I2C0_SCL
- U3 pad 15: (no net) -> I2C0_SDA
- U3 pad 16: (no net) -> TS_BIAS
- U3 pad 17: (no net) -> ILIM_SET
- U3 pad 18: (no net) -> BATT_F
- U3 pad 2: GND -> VBUS_IN
- U3 pad 20: (no net) -> PROG_SET
- U3 pad 21: (no net) -> GPIO_CHG_INT
- U3 pad 22: (no net) -> BATT_F
- U3 pad 23: (no net) -> BATT_F
- U3 pad 25: (no net) -> SYS_NODE
- U3 pad 3: CHG_SW -> VBUS_IN
- U3 pad 4: +3V3 -> BTST1
- U3 pad 5: I2C0_SDA -> REGN
- U3 pad 6: I2C0_SCL -> (no net)
- U3 pad 7: PROG -> (no net)
- U3 pad 9: (no net) -> DOCK_OK
Routing:
- net Q5_Q6_MID: track 0.00 -> 61.8 mm
- net +5V0: track 0.00 -> 56.9 mm
- net BOOT_5V: track 0.00 -> 29.5 mm
- net BATT_F: track 0.00 -> 29.2 mm
- net VBUS_IN: track 0.00 -> 21.4 mm
- net FB5V: track 0.00 -> 17.9 mm
- net VBAT_P1_OUT: track 0.00 -> 17.4 mm
- net +3V3: track 0.00 -> 14.5 mm
- net DOCK_F: track 0.00 -> 13.4 mm
- net DOCK_OK: track 0.00 -> 12.6 mm
- net P1_F: track 0.00 -> 4.20 mm
