File: Maverick1000/kicad/SKYWARD-COMPUTE-CARRIER/SKYWARD-COMPUTE-CARRIER.kicad_sch (KiCad schematic)
At the start: 75 parts, among them J1 CM4_J1, J10 DEBUG, J2 CM4_J2, J3 BATT_IN, J4 DOCK, J5 FC, J6 GNSS, J7 ELRS, J8 TOF, J9 TERRA, Q1 SQJ438EP, Q2 SQJ438EP, SW1 nRPIBOOT, SW2 RUN, U1 LM74610QDBVRQ1, U2 LM74610QDBVRQ1, U3 BQ25792RQMR, U4 TPS5430DDA, U5 AP2112K-3.3TRG1, U6 INA3221AIPW

Commit message: Audit SKYWARD-COMPUTE-CARRIER Rev A: verify against real datasheets, run real DRC, route priority nets, fix defects found
Full engineering audit pass per the fabrication-readiness review brief.
Re-verified every real component against authoritative sources instead of
trusting the existing netlist, and fixed what was found broken rather than
routing around it:

- CM4 J1/J2 pin numbers and footprint (DF40C-100DS-0.4V pad numbering was
  sequential instead of the real odd/even scheme -- would have produced a
  non-functional board), plus a UART-availability architecture error
  (assumed 5 independent UARTs, only 3 are actually usable)
- BQ25792 charger fully re-modeled from a fictional 8-pin part to the real
  29-pin WQFN 4-switch buck-boost topology, with a complete verified
  application circuit
- LM74610 ORing controller corrected from an invented 6-pin package to the
  real 8-pin VSSOP-8 (no GND pin, floats between ANODE/CATHODE)
- P-FET part number "SQJ438EP" was not a real, findable part; replaced
  with verified-real DMP2305U-7
- CM4 J2 schematic symbol was reusing J1's pin labels (net wiring was
  correct, displayed pin names were wrong for ~half of J2's pins) -- found
  via an ERC-equivalent netlist check, fixed with a distinct J2 symbol
- U4 (TPS5430 5V buck) was missing its catch diode entirely -- confirmed
  non-synchronous via 6 independent reference designs, fixed by adding D5

Ran real KiCad DRC (pcbnew.WriteDRCReport, since this KiCad 7.0.11 build
has no CLI erc/drc subcommands) and used it to find and fix two more real
bugs: a collision-checker bug in this project's own router that had
wrongly certified some tracks as short-free when they actually crossed a
different net, and a BQ25792 footprint exposed-pad overlapping real pins.

Routed the 59 highest-priority nets (battery/converter/charging paths)
with a verified point-to-point router: 13 succeeded as real, DRC-clean
copper; 46 remain ratsnest, including every power-converter switch node.
Zone filli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
Parts:
- removed J1: CM4_J1, SKYWARD_Custom:Hirose_DF40C-100DS-0.4V, symbol SKYWARD_Custom:CM4_Connector_100
- removed J2: CM4_J2, SKYWARD_Custom:Hirose_DF40C-100DS-0.4V, symbol SKYWARD_Custom:CM4_Connector_100
- removed U1, U2: LM74610QDBVRQ1, Package_TO_SOT_SMD:SOT-23-6, symbol SKYWARD_Custom:LM74610
- removed U3: BQ25792RQMR, Package_DFN_QFN:QFN-24-1EP_4x4mm_P0.5mm_EP2.6x2.6mm, symbol SKYWARD_Custom:BQ25792
- added C21: 10uF, Capacitor_SMD:C_0805_2012Metric, symbol Device:C
- added C22: 100nF, Capacitor_SMD:C_0402_1005Metric, symbol Device:C
- added D5: SS34, Diode_SMD:D_SMA, symbol Device:D_Schottky
- added J1: CM4_J1, SKYWARD_Custom:Hirose_DF40C-100DS-0.4V, symbol SKYWARD_Custom:CM4_Connector_100_J1
- added J2: CM4_J2, SKYWARD_Custom:Hirose_DF40C-100DS-0.4V, symbol SKYWARD_Custom:CM4_Connector_100_J2
- added Q5, Q6: DMP2305U-7, Package_TO_SOT_SMD:SOT-23, symbol Device:Q_PMOS_GSD
- added R16: 5.6k, Resistor_SMD:R_0402_1005Metric, symbol Device:R
- added R17, R18, R20, R21: 10k, Resistor_SMD:R_0402_1005Metric, symbol Device:R
- added R19: 10, Resistor_SMD:R_0402_1005Metric, symbol Device:R
- added U1, U2: LM74610QDGKRQ1, Package_SO:VSSOP-8_3.0x3.0mm_P0.65mm, symbol SKYWARD_Custom:LM74610QDGKRQ1
- added U3: BQ25792RQMR, SKYWARD_Custom:QFN-29_L4.0-W4.0-P0.40-BQ25792RQMR, symbol SKYWARD_Custom:BQ25792RQMR
- C10: value 100nF -> 10uF; footprint Capacitor_SMD:C_0402_1005Metric -> Capacitor_SMD:C_0805_2012Metric
- C9: value 100nF -> 1uF; footprint Capacitor_SMD:C_0402_1005Metric -> Capacitor_SMD:C_0603_1608Metric
- Q1, Q2: value SQJ438EP -> DMP2305U-7
Connections:
- net UART3_RXD is gone; now on net UART0_RXD0: J10.4 (Pin_4)
- net UART3_TXD is gone; now on net UART0_TXD0: J10.3 (Pin_3)
- net +3V3: now also J1.99 (+3V3), R20.1, R21.1; no longer C10.1, C9.1
- net +5V0: now also J1.77 (+5V0), J1.79 (+5V0), J1.81 (+5V0), J1.83 (+5V0), J1.85 (+5V0), J1.87 (+5V0)
- net 5V0_SW: now also D5.1 (K)
- net BATT_F: now also C21.1, U1.4 (ANODE), U3.18 (BATP), U3.22 (BAT), U3.23 (BAT); no longer C8.1, L2.2
- net DOCK_OK: now also C22.2, Q5.2 (S), U3.9 (VAC1); no longer C7.1
- net EEPROM_nWP: now also J1.20 (EEPROM_nWP)
- net GND: now also C21.2, D5.2 (A), J1.1 (GND), J1.13 (GND), J1.14 (GND), J1.2 (GND), J1.22 (GND), J1.23 (GND), J1.32 (GND), J1.33 (GND), J1.42 (GND), J1.43 (GND), J1.52 (GND), J1.53 (GND), J1.59 (GND), J1.60 (GND), J1.65 (GND), J1.66 (GND), J1.7 (GND), J1.71 (GND), J1.74 (GND), J1.8 (GND), J1.98 (GND), J2.1 (GND), J2.13 (GND), J2.14 (GND), J2.19 (GND), J2.20 (GND), J2.25 (GND), J2.26 (GND), J2.7 (GND), J2.8 (GND), R16.2, R18.2, U3.13 (~{CE}), U3.27 (GND), U3.30 (EP), U3.8 (VAC2); no longer C16.2, C17.2
- net GPIO_DOCK_DET: now also J1.30 (GPIO_DOCK_DET)
- net GPIO_FC_AUX: now also J1.47 (GPIO_FC_AUX)
- net GPIO_FC_RESET: now also J1.46 (GPIO_FC_RESET)
- net GPIO_GNSS_PPS: now also J1.29 (GPIO_GNSS_PPS)
- net GPIO_STATUS_LED: now also J1.45 (GPIO_STATUS_LED)
- net GPIO_TERRA_A: now also J1.27 (GPIO_TERRA_A)
- net GPIO_TERRA_B: now also J1.25 (GPIO_TERRA_B)
- net GPIO_TERRA_IRQ: now also J1.49 (GPIO_TERRA_IRQ)
- net GPIO_TERRA_TRIG: now also J1.26 (GPIO_TERRA_TRIG)
- net GPIO_TOF_INT: now also J1.50 (GPIO_TOF_INT)
- net I2C0_SCL: now also J1.35 (I2C0_SCL), U3.14 (SCL)
- net I2C0_SDA: now also J1.36 (I2C0_SDA), U3.15 (SDA)
- net P1_F: now also U2.4 (ANODE)
- net Q1_GATE: now also U1.2 (GATE_PULL_DOWN), U1.6 (GATE_DRIVE)
- net Q2_GATE: now also U2.2 (GATE_PULL_DOWN), U2.6 (GATE_DRIVE)
- net SPI0_CE0_N: now also J1.39 (SPI0_CE0_N)
- net SPI0_MISO: now also J1.40 (SPI0_MISO)
- net SPI0_MOSI: now also J1.44 (SPI0_MOSI)
- net SPI0_SCLK: now also J1.38 (SPI0_SCLK)
- net UART0_RXD0: now also J1.51 (UART0_RXD0)
- net UART0_TXD0: now also J1.55 (UART0_TXD0)
- net USB2_0_DN: now also J2.3 (USB2_0_DN)
- net USB2_0_DP: now also J2.5 (USB2_0_DP)
- net VBAT_MAIN_OUT: now also U1.8 (CATHODE)
- net VBAT_P1_OUT: now also U2.8 (CATHODE)
- net nRPIBOOT: now also J1.93 (nRPIBOOT)
- net CHG_SW renamed SW1
- net SW1: now also U3.28 (SW1)
- net PROG renamed ILIM_SET
- net ILIM_SET: now also U3.17 (ILIM_HIZ)
- net RUN_PG_N renamed RUN_PG
- net RUN_PG: now also J1.92 (RUN_PG)
- net UART1_RXD1 renamed UART3_RXD3
- net UART3_RXD3: now also J1.34 (UART3_RXD3)
- net UART1_TXD1 renamed UART3_TXD3
- net UART3_TXD3: now also J1.54 (UART3_TXD3)
- net UART2_RXD renamed UART5_RXD5
- net UART5_RXD5: now also J1.28 (UART5_RXD5)
- net UART2_TXD renamed UART5_TXD5
- net UART5_TXD5: now also J1.31 (UART5_TXD5)
- net UART4_RXD: no longer names the net of J9.11 (NC)
- net UART4_TXD: no longer names the net of J9.10 (NC)
- net VCAP1 renamed VCAP1_L
- net VCAP1_L: now also U1.1 (VCAPL)
- net VCAP2 renamed VCAP2_L
- net VCAP2_L: now also U2.1 (VCAPL)
- new net ACDRV1_GATE: R19.1, U3.11 (ACDRV1)
- new net BTST1: C22.1, U3.4 (BTST1)
- new net GATE_DRIVE: Q5.1 (G), Q6.1 (G), R19.2
- new net GPIO_CHG_INT: J1.24 (GPIO_CHG_INT), R21.2, U3.21 (~{INT})
- new net PMID: C10.1, U3.29 (PMID)
- new net PROG_SET: R16.1, U3.20 (PROG)
- new net Q5_Q6_MID: Q5.3 (D), Q6.3 (D)
- new net QON_N: R20.2, U3.12 (~{QON})
- new net REGN: C9.1, R17.1, U3.5 (REGN)
- new net SW2: L2.2, U3.26 (SW2)
- new net SYS_NODE: C8.1, U3.25 (SYS)
- new net TS_BIAS: R17.2, R18.1, U3.16 (TS)
- new net VBUS_IN: C7.1, Q6.2 (S), U3.2 (VBUS), U3.3 (VBUS)
- new net VCAP1_H: C16.2, U1.7 (VCAPH)
- new net VCAP2_H: C17.2, U2.7 (VCAPH)
- no-connect marks 155 -> 157
