File: Maverick1000/kicad/SKYWARD-COMPUTE-CARRIER/SKYWARD-COMPUTE-CARRIER.kicad_sch (KiCad schematic)
At the start: 118 parts, among them J1 CM4_J1, J10 DEBUG, J11 SIM_TRAY, J12 ANT_CELLULAR, J13 USB_BOOT, J2 CM4_J2, J3 BATT_IN, J4 DOCK, J5 FC, J6 GNSS, J7 ELRS, J8 TOF, J9 TERRA, Q1 DMP2305U-7, Q2 DMP2305U-7, Q5 DMP2305U-7, Q6 DMP2305U-7, SW1 nRPIBOOT, SW2 RUN, U1 LM74610QDGKRQ1, U10 FSUSB42MUX, U2 LM74610QDGKRQ1, U3 BQ25792RQMR, U4 TPS5430DDA, U5 AP2112K-3.3TRG1, U6 INA3221AIPW, U7 USB2512B-AEZG-TR, U8 EC25VFA-512-STD, U9 TPS5430DDA, Y1 24MHz

Commit message: Rename company Frontier Robotics/Industries -> Frontier Innovations
Applied consistently across every instance: KiCad schematic/PCB source
(including the board's own silkscreen text and the three Python
generator scripts that produce it, so regeneration won't reintroduce
the old name), exported netlists, and docs. Re-verified after the
rename with real tooling, not just trusted:

- Re-rendered the board's silkscreen (kicad-cli, --exclude-drawing-
  sheet) and visually confirmed "FRONTIER INNOVATIONS" is centered and
  clear of the mounting-hole labels on both edges, no overflow.
- Re-ran python/run_drc.py: still 0 unconnected pads, same 2 pre-
  existing/documented lib_footprint_mismatch warnings, nothing new.
- Re-ran the netlist cross-check against a fresh kicad-cli export:
  still 0 mismatches, 469/469.
- Regenerated the two manufacturing preview SVGs that still had the
  old name baked into their rendered text.

Left one historical quote in docs/FINAL_DESIGN_AUDIT.md untouched
(a past session's note describing a stale "FRONTIER ROBOTICS" board
silkscreen bug it found and fixed) since rewriting it would make that
history inaccurate, not more correct.

Co-Authored-By: Claude Sonnet 5 <noreply@anthropic.com>
Claude-Session: https://claude.ai/code/session_01PjVLbuUxJUCeC3xm5gJT9X
Other:
- company: Frontier Industries -> Frontier Innovations
Changed lines of the file:
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@@
     (date "2026-09-21")
     (rev "A")
-    (company "Frontier Industries")
+    (company "Frontier Innovations")
     (comment 1 "Internal codename: SKYWARD. Product: Maverick 1000.")
     (comment 2 "See docs/assumptions.md before fabrication -- CM4 pinout and DF40C footprint need datasheet verification.")
